Commit message: Add reachable points computation in estimate.ipynb ,add reachable points config file, update mouting plate position in urdf to be less convoluted

File: src/rr100_ur_description/urdf/rr100_ur.urdf.xacro (robot description, xacro)
@@ -1,6 +1,4 @@
 <?xml version="1.0"?>
 <robot xmlns:xacro="http://www.ros.org/wiki/xacro" name="chassis">
-    <xacro:include filename="$(find rr100_description)/urdf/rr100.urdf.xacro" />
-    <xacro:include filename="$(find ur5e_gripper_description)/urdf/ur_hand_e.xacro" />
     <!-- Base Size -->
     <xacro:property name="chassis_x_size" value="0.80" />
@@ -12,6 +10,9 @@
     <xacro:property name="plate_width" value="0.25" />
     <xacro:property name="plate_height" value="0.2" />
+    <!-- Actual value -->
     <xacro:property name="plate_thickness" value="0.01" />
-    <xacro:property name="rail_size" value="0.02" />
+     <!-- Elevated value -->
+    <!-- <xacro:property name="plate_thickness" value="0.40" />  -->
+    <xacro:property name="rail_size" value="0.025" />
     <xacro:property name="M_PI" value="3.14159" />
     <!-- parameters -->
@@ -29,18 +30,26 @@
     <xacro:arg name="safety_k_position" default="20" />
     <xacro:arg name="ur_prefix" default="ur_"/>
+    <xacro:include filename="$(find rr100_description)/urdf/rr100.urdf.xacro" />
+    <xacro:include filename="$(find ur5e_gripper_description)/urdf/ur_hand_e.xacro" />
     <link name="mounting_base_link">
         <visual>
             <origin xyz="0 0 0" rpy="0 0 ${M_PI / 2}" />
             <geometry>
+                <!-- Actual -->
                 <mesh filename="package://rr100_ur_description/meshes/ur5_mounting_plate.stl"
                     scale="0.001 0.001 0.001" />
+                <!-- Elevated -->
+                <!-- <mesh filename="package://rr100_ur_description/meshes/ur5_mounting_plate_shifted.stl"
+                    scale="0.001 0.001 0.04" /> -->
             </geometry>
             <material name="grey" />
         </visual>
         <collision>
-            <origin xyz="0 0 0" rpy="0 0 0" />
+            <origin xyz="0 0 0" rpy="0 0 ${M_PI / 2}" />
             <geometry>
+                <!-- Actual -->
                 <mesh filename="package://rr100_ur_description/meshes/ur5_mounting_plate.stl"
                     scale="0.001 0.001 0.001" />
+                <!-- <box size="${plate_width} ${plate_height} ${plate_thickness}"/> -->
             </geometry>
         </collision>
@@ -49,11 +58,10 @@
         <!-- ${-base_x_size/2 + 0.025 + 0.2 / 2} 0 ${base_z_size} -->
         <origin
-            xyz="${-chassis_x_size/2 + plate_rear_distance + plate_height / 2} 0 ${(base_z_size + ground_clearance) / 2 + plate_thickness + plate_thickness / 2 + rail_size}"
+            xyz="${-chassis_x_size/2 + plate_rear_distance + plate_height / 2} 0 ${(base_z_size + ground_clearance) / 2 + plate_thickness / 2 + rail_size}"
             rpy="0 0 0" />
         <parent link="base_link" />
         <child link="mounting_base_link" />
     </joint>
-    <gazebo reference="mounting_base_link">
-    </gazebo>
+    <gazebo reference="mounting_base_link"/>
     <xacro:ur5_hand_e
         prefix="$(arg ur_prefix)"
@@ -67,4 +75,7 @@
         safety_k_position="$(arg safety_k_position)" />
     <joint name="ur_base_joint" type="fixed">
+        <origin
+            xyz="0 0 ${plate_thickness / 2}"
+            rpy="0 0 0" />
         <parent link="mounting_base_link"/>
         <child link="$(arg ur_prefix)base_link"/>

Commit message: Add aruco localizer node, readme.md

File: src/rr100_ur_description/urdf/rr100_ur.urdf.xacro (robot description, xacro)
@@ -7,10 +7,10 @@
     <xacro:property name="ground_clearance" value="0.11" />
     <!-- Mounting plate properties (in meters)-->
-    <xacro:property name="plate_rear_distance" value="0.05"/>
+    <xacro:property name="plate_rear_distance" value="0.05" />
     <xacro:property name="plate_width" value="0.25" />
     <xacro:property name="plate_height" value="0.2" />
     <!-- Actual value -->
     <xacro:property name="plate_thickness" value="0.01" />
-     <!-- Elevated value -->
+    <!-- Elevated value -->
     <!-- <xacro:property name="plate_thickness" value="0.40" />  -->
     <xacro:property name="rail_size" value="0.025" />
@@ -29,5 +29,5 @@
     <xacro:arg name="safety_pos_margin" default="0.15" />
     <xacro:arg name="safety_k_position" default="20" />
-    <xacro:arg name="ur_prefix" default="ur_"/>
+    <xacro:arg name="ur_prefix" default="ur_" />
     <xacro:include filename="$(find rr100_description)/urdf/rr100.urdf.xacro" />
     <xacro:include filename="$(find ur5e_gripper_description)/urdf/ur_hand_e.xacro" />
@@ -40,5 +40,6 @@
                     scale="0.001 0.001 0.001" />
                 <!-- Elevated -->
-                <!-- <mesh filename="package://rr100_ur_description/meshes/ur5_mounting_plate_shifted.stl"
+                <!-- <mesh
+                filename="package://rr100_ur_description/meshes/ur5_mounting_plate_shifted.stl"
                     scale="0.001 0.001 0.04" /> -->
             </geometry>
@@ -63,5 +64,13 @@
         <child link="mounting_base_link" />
     </joint>
-    <gazebo reference="mounting_base_link"/>
+    <link name="aruco_marker_link" />
+    <joint name="aruco_marker_joint" type="fixed">
+        <origin
+            xyz="0 0 0.0807"
+            rpy="0 0 0" />
+        <parent link="rslidar_base_link" />
+        <child link="aruco_marker_link" />
+    </joint>
+    <gazebo reference="mounting_base_link" />
     <xacro:ur5_hand_e
         prefix="$(arg ur_prefix)"
@@ -78,6 +87,6 @@
             xyz="0 0 ${plate_thickness / 2}"
             rpy="0 0 0" />
-        <parent link="mounting_base_link"/>
-        <child link="$(arg ur_prefix)base_link"/>
+        <parent link="mounting_base_link" />
+        <child link="$(arg ur_prefix)base_link" />
     </joint>
 </robot>

Commit message: Add urdf output option to rr100_ur_description

File: src/rr100_ur_description/urdf/rr100_ur.urdf.xacro (robot description, xacro)
@@ -30,4 +30,7 @@
     <xacro:arg name="safety_k_position" default="20" />
     <xacro:arg name="ur_prefix" default="ur_" />
+    <xacro:arg name="rslidar_enabled" default="true" />
+    <xacro:arg name="realsense_enabled" default="true" />
+    <xacro:arg name="gps_enabled" default="true" />
     <xacro:include filename="$(find rr100_description)/urdf/rr100.urdf.xacro" />
     <xacro:include filename="$(find ur5e_gripper_description)/urdf/ur_hand_e.xacro" />
@@ -64,12 +67,14 @@
         <child link="mounting_base_link" />
     </joint>
-    <link name="aruco_marker_link" />
-    <joint name="aruco_marker_joint" type="fixed">
-        <origin
-            xyz="0 0 0.073"
-            rpy="0 0 0" />
-        <parent link="rslidar_base_link" />
-        <child link="aruco_marker_link" />
-    </joint>
+    <xacro:if value="$(arg rslidar_enabled)">
+        <link name="aruco_marker_link" />
+        <joint name="aruco_marker_joint" type="fixed">
+            <origin
+                xyz="0 0 0.073"
+                rpy="0 0 0" />
+            <parent link="rslidar_base_link" />
+            <child link="aruco_marker_link" />
+        </joint>
+    </xacro:if>
     <gazebo reference="mounting_base_link" />
     <xacro:ur5_hand_e
